File: SvayamV3_IIK.kicad_pcb (KiCad board)
At the start: 6 copper layers, 125.1 x 90 mm, 290 parts, among them J1 USB_C_Receptacle_USB2.0_16P, J10 Micro_SD_Card_Det1, J11 BUZZER, J12 ADC, J13 CAN, J14 SERIAL5, J15 SAFETY, J16 POWER2, J17 I2C, J18 CAN2, J19 Channel 1, J2 GPS, J20 Channel 5, J21 Channel 9, J22 Channel 13, J23 Channel 2, J24 Channel 6, J25 Channel 10, J26 Channel 14, J27 Channel 3, J28 Channel 7, J29 Channel 11, J3 SPI, J30 Channel 15, J31 Channel 4, J32 Channel 8, J33 Channel 12, J34 Channel 16, J4 TELEM1, J5 TELEM2, J6 SBUS, J7 Conn_01x05_Pin, J8 SERIAL4, J9 POWER1, Q1 AO3400A, SW1 SK-3296S-01-L3, SW2 TS-1010A-B, U1 STM32H743IIK6, U10 TPS2120YFPR, U11 TPS63070, U12 RT9080-33GJ5, U13 RT9080-33GJ5, U14 AP22804AW5, U15 USBLC6-2SC6, U16 TPS2553DBVT, U17 TPS2553DBVT, U18 TPS2553DBVT, U19 TPS2553DBVT, U2 FM25CL64B, U20 TPS2553DBVT, U21 TPS2553DBVT, U22 TPS2553DBVT, U23 TPS2553DBVT, U24 TPS2553DBVT, U3 TJA1051TK-3, U4 TJA1051TK-3, U5 BMP388, U6 DPS310XTSA1, U7 BMI088, U8 BMI270, U9 BMM150, Y1 X50328MSB2GI

Commit message: PCB: 3 via GND keluar dari pad MP (J17 kanan, J11) — DRC 760->752, short nyata 0
Fungsi: unconnected 0, parity 0, short antar dua net nyata 0. 2 shorting_items sisa
adalah via +5V_PERIPH di dalam pad MP kiri J17 (MP tanpa net -> bukan short aktif,
tapi jadi +5V-GND kalau MP di-assign GND sebelum via dipindah).

Perubahan angka (23:28 -> 23:35):
- shorting_items 5 -> 2        solder_mask_bridge 17 -> 14
- hole_clearance 24 -> 22      hole_to_hole 15 -> 14
- clearance 27 -> 28 (+1, area fanout BGA)
- total 760 -> 752 (313 error / 439 warning)

Docs: README + STATUS.md disinkronkan; docs/reports + docs/board-stats.txt di-refresh.
Verifikasi: kicad-cli 10.0.6 pcb drc --severity-all --schematic-parity
Routing:
- net GND: track 463.9 -> 465.5 mm
Changed lines of the file:
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@@
-	)
-	(segment
-		(start 104.021178 146.071178)
-		(end 104.936178 146.071178)
-		(width 0.2)
-		(layer "F.Cu")
-		(net "GND")
 	)
 	(segment
@@
 	)
 	(segment
+		(start 104.031178 146.061178)
+		(end 104.021178 146.071178)
+		(width 0.5)
+		(layer "F.Cu")
+		(net "GND")
+	)
+	(segment
 		(start 105.86 99.393499)
 		(end 105.86 99.881)
@@
 	)
 	(segment
+		(start 105.526178 146.071178)
+		(end 105.536178 146.061178)
+		(width 0.2)
+		(layer "F.Cu")
+		(net "GND")
+	)
+	(segment
 		(start 99.06444 131.53944)
 		(end 99.721178 130.882701)
@@
 	)
 	(segment
+		(start 102.507678 146.04)
+		(end 103.99 146.04)
+		(width 0.5)
+		(layer "F.Cu")
+		(net "GND")
+	)
+	(segment
 		(start 99.296178 130.396178)
 		(end 99.296178 130.457701)
@@
 	)
 	(segment
+		(start 102.538856 146.071178)
+		(end 102.507678 146.04)
+		(width 0.2)
+		(layer "F.Cu")
+		(net "GND")
+	)
+	(segment
 		(start 103.439 106.881)
 		(end 103.2325 107.0875)
@@
 	)
 	(segment
+		(start 105.536178 146.061178)
+		(end 104.031178 146.061178)
+		(width 0.5)
+		(layer "F.Cu")
+		(net "GND")
+	)
+	(segment
 		(start 100.92 108.73625)
 		(end 100.56 108.37625)
@@
 	)
 	(segment
+		(start 103.99 146.04)
+		(end 104.021178 146.071178)
+		(width 0.5)
+		(layer "F.Cu")
+		(net "GND")
+	)
+	(segment
 		(start 100.640417 131.80194)
 		(end 98.801939 133.640418)
@@
 	)
 	(segment
-		(start 104.936178 146.071178)
-		(end 105.526178 146.071178)
-		(width 0.2)
-		(layer "F.Cu")
-		(net "GND")
-	)
-	(segment
 		(start 64.85 144.025)
 		(end 66.175 145.35)
@@
 	)
 	(segment
-		(start 105.526178 146.071178)
-		(end 105.536178 146.061178)
-		(width 0.2)
-		(layer "F.Cu")
-		(net "GND")
-	)
-	(segment
 		(start 105.3075 106.406)
 		(end 105.4825 106.231)
@@
 	)
 	(via
-		(at 104.936178 146.071178)
+		(at 102.507678 146.04)
 		(size 0.6)
 		(drill 0.3)
@@
 	)
 	(via
-		(at 89.155 135.1)
+		(at 87.882 134.5)
 		(size 0.7)
 		(drill 0.3)
@@
 	)
 	(via
-		(at 89.0525 135.6)
-		(size 0.7)
-		(drill 0.3)
+		(at 87.882 135.152918)
+		(size 0.7)
+		(drill 0.3)
